File: Telemetria_Hardware.kicad_pcb (KiCad board)
At the start: 2 copper layers, 81.3 x 87.6 mm, 16 parts, among them M100A 1715734

Commit message: placa teste
Parts:
- removed B150A, M100A: 1715734, Terminal_Block_PCB_3Way:Connector_KRE_3W_5,08mm
- removed DHT: Conn_01x04_Female, Connector_PinSocket_2.54mm:PinSocket_1x04_P2.54mm_Vertical
- removed MPPT, STEP: CTB1202_2BK, Terminal_Block_PCB_2Way:KRE_Terminal_2Way_5.08mm
- added ?: , , F.Cu at (76.2, 134.6)
- added ?: , , F.Cu at (81.3, 134.6)
- added ACS3: Conn_01x03_Female, Connector_PinSocket_2.54mm:PinSocket_1x03_P2.54mm_Vertical, F.Cu at (142.2, 96.5)
- added B150A1: 1715734, TerminalBlock:TerminalBlock_bornier-3_P5.08mm, F.Cu at (116.8, 53.3)
- added DHT1: Conn_01x04_Female, Connector_PinSocket_2.54mm:PinSocket_1x04_P2.54mm_Vertical, F.Cu at (86.4, 124.5)
- added M100A1: 1715734, TerminalBlock:TerminalBlock_bornier-3_P5.08mm, F.Cu at (94.0, 53.3)
- added MPPT1: CTB1202_2BK, TerminalBlock:TerminalBlock_bornier-2_P5.08mm, F.Cu at (73.7, 114.3)
- added PCB_Vin2: CTB1202_2BK, TerminalBlock:TerminalBlock_bornier-2_P5.08mm, F.Cu at (124.5, 144.8)
- added PCB_Vin3: CTB1202_2BK, TerminalBlock:TerminalBlock_bornier-2_P5.08mm, F.Cu at (109.2, 144.8)
- added R10: R, Resistor_THT:R_Axial_DIN0207_L6.3mm_D2.5mm_P10.16mm_Horizontal, F.Cu at (112.8, 121.9)
- added R11: R, Resistor_THT:R_Axial_DIN0207_L6.3mm_D2.5mm_P10.16mm_Horizontal, F.Cu at (106.7, 121.9)
- added R5: R, Resistor_THT:R_Axial_DIN0207_L6.3mm_D2.5mm_P10.16mm_Horizontal, F.Cu at (139.7, 101.6)
- added R6: R, Resistor_THT:R_Axial_DIN0207_L6.3mm_D2.5mm_P10.16mm_Horizontal, F.Cu at (149.9, 101.6)
- added R7: R, Resistor_THT:R_Axial_DIN0207_L6.3mm_D2.5mm_P10.16mm_Horizontal, F.Cu at (88.9, 132.1)
- added R8: R, Resistor_THT:R_Axial_DIN0207_L6.3mm_D2.5mm_P10.16mm_Horizontal, F.Cu at (124.5, 121.9)
- added R9: R, Resistor_THT:R_Axial_DIN0207_L6.3mm_D2.5mm_P10.16mm_Horizontal, F.Cu at (119.4, 121.9)
- added STEP1: CTB1202_2BK, TerminalBlock:TerminalBlock_bornier-2_P5.08mm, F.Cu at (142.2, 121.9)
- PCB_Vin1: footprint Terminal_Block_PCB_2Way:KRE_Terminal_2Way_5.08mm -> TerminalBlock:TerminalBlock_bornier-2_P5.08mm
- moved C1 7.18 mm to (134.6, 124.5), turned to 180 degrees
- moved C2 2.54 mm to (77.5, 124.5)
Connections:
- ACS1 pad 2: Net-(ACS1-Pad2) -> Net-(ACS1-Pin_2)
- ACS2 pad 2: Net-(ACS2-Pad2) -> Net-(ACS2-Pin_2)
- ADS1115 pad 1: Net-(C2-Pad1) -> Net-(ADS1115-VDD)
- ADS1115 pad 3: Net-(ADS1115-Pad3) -> Net-(ADS1115-SCL)
- ADS1115 pad 4: Net-(ADS1115-Pad4) -> Net-(ADS1115-SDA)
- C2 pad 1: Net-(C2-Pad1) -> Net-(ADS1115-VDD)
- ESP32 pad 12: unconnected-(ESP32-Pad12) -> Net-(ESP32-IO12)
- ESP32 pad 13: unconnected-(ESP32-Pad13) -> Net-(ESP32-IO13)
- ESP32 pad 7: unconnected-(ESP32-Pad7) -> Net-(ESP32-IO33)
- R1 pad 1: Net-(ESP32-Pad21) -> Net-(ESP32-IO16)
- R2 pad 2: Net-(ESP32-Pad21) -> Net-(ESP32-IO16)
Routing:
- net Net-(ACS1-Pin_1): track 129.5 -> 178.0 mm
- net Net-(ESP32-IO33): track 0.00 -> 47.8 mm
- net Net-(ESP32-IO12): track 0.00 -> 35.3 mm
- net Net-(ESP32-IO13): track 0.00 -> 26.9 mm
- net GND: track 23.4 -> 0.00 mm
- net Net-(ADS1115-VDD): track 0.00 -> 17.5 mm
- net Net-(PCB_Vin2-Pad1): track 0.00 -> 14.8 mm
- net Net-(PCB_Vin3-Pad1): track 0.00 -> 13.8 mm
- net Net-(ACS3-Pin_2): track 0.00 -> 9.38 mm
- net Net-(ADS1115-A0): track 51.8 -> 56.9 mm
- net Net-(ADS1115-A1): track 40.8 -> 45.7 mm
- net Net-(C2-Pad1): track 106.7 -> 101.9 mm
Other:
- board outline removed
- board text removed: "Telemeteam Agatti Raibolt Fernando"

Commit message: teste 2
Parts:
- removed ? (x2): , 
- removed C2: C_Polarized, Capacitor_THT:C_Radial_D6.3mm_H11.0mm_P2.50mm
- removed DHT1: Conn_01x04_Female, Connector_PinSocket_2.54mm:PinSocket_1x04_P2.54mm_Vertical
- removed R7: R, Resistor_THT:R_Axial_DIN0207_L6.3mm_D2.5mm_P10.16mm_Horizontal
- added R12: R, Resistor_THT:R_Axial_DIN0207_L6.3mm_D2.5mm_P10.16mm_Horizontal, F.Cu at (99.1, 109.2)
- added SW1: RESET BUTTON, BUTT:BUTT, F.Cu at (91.4, 97.8)
- ESP32: footprint esp32_devkit_v1_doit:esp32_devkit_v1_doit -> ESP32:esp32_devkit_v1_doit
- moved R8 37.0 mm to (87.6, 118.1), turned to 0 degrees
- moved R9 31.8 mm to (87.6, 123.2), turned to 0 degrees
- moved R10 26.3 mm to (87.6, 129.5), turned to 0 degrees
- moved R11 23.5 mm to (87.6, 135.7), turned to 0 degrees
- moved B150A1 23.2 mm to (94.0, 57.1)
- moved M100A1 20.7 mm to (73.7, 57.1)
- moved R1 20.5 mm to (95.2, 91.4)
- moved R2 20.5 mm to (85.1, 86.4)
- moved R4 20.5 mm to (95.2, 73.7)
- moved R3 20.5 mm to (95.2, 81.3)
- moved STEP1 13.1 mm to (148.6, 133.3), turned to 180 degrees
- moved ADS1115 12.9 mm to (75.9, 66.0)
- moved PCB_Vin2 11.7 mm to (121.9, 133.3)
- moved PCB_Vin3 11.7 mm to (106.7, 133.3)
- moved C1 7.72 mm to (135.8, 132.1)
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Connections:
- ESP32 pad 16: Net-(C2-Pad1) -> Net-(ADS1115-VDD)
- ESP32 pad 18: Net-(DHT1-Pad2) -> unconnected-(ESP32-IO15-Pad18)
- ESP32 pad 20: unconnected-(ESP32-Pad20) -> Net-(ADS1115-VDD)
- ESP32 pad 21: Net-(ESP32-Pad21) -> Net-(ESP32-IO16)
- ESP32 pad 26: Net-(ADS1115-Pad4) -> Net-(ADS1115-SDA)
- ESP32 pad 29: Net-(ADS1115-Pad3) -> Net-(ADS1115-SCL)
- ESP32 pad 4: Net-(ACS1-Pad2) -> Net-(ACS1-Pin_2)
- ESP32 pad 5: Net-(ACS2-Pad2) -> Net-(ACS2-Pin_2)
- ESP32 pad 6: unconnected-(ESP32-Pad6) -> GND
Routing:
- net GND: track 0.00 -> 193.8 mm
- net Net-(C2-Pad1): track 101.9 -> 0.00 mm
- net Net-(ADS1115-VDD): track 17.5 -> 104.6 mm
- net Net-(ESP32-IO12): track 35.3 -> 73.0 mm
- net Net-(ADS1115-SDA): track 0.00 -> 36.3 mm
- net Net-(ADS1115-SCL): track 0.00 -> 31.6 mm
- net Net-(ACS2-Pad2): track 30.5 -> 0.00 mm
- net Net-(DHT1-Pad2): track 30.4 -> 0.00 mm
- net Net-(ACS1-Pad2): track 30.1 -> 0.00 mm
- net Net-(ACS1-Pin_2): track 0.00 -> 29.7 mm
- net Net-(ESP32-IO13): track 26.9 -> 56.1 mm
- net Net-(ESP32-Pad21): track 24.9 -> 0.00 mm
- net Net-(ADS1115-Pad4): track 22.1 -> 0.00 mm
- net Net-(ACS2-Pin_2): track 0.00 -> 18.9 mm
- net Net-(PCB_Vin1-Pad1): track 8.93 -> 27.0 mm
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
Commit message: teste 3
Parts:
- moved R4 10.2 mm to (85.1, 74.9), turned to 0 degrees
- moved MPPT1 8.13 mm to (71.1, 120.7)
- moved PCB_Vin1 6.35 mm to (72.4, 105.4)
- moved R10 4.02 mm to (88.9, 133.3)
- moved R11 4.02 mm to (88.9, 139.5)
- moved R9 4.02 mm to (88.9, 127.0)
- moved R8 2.84 mm to (88.9, 120.7)
- moved ACS3 1.88 mm to (144.1, 96.5)
Connections:
- ESP32 pad 5: Net-(ACS2-Pin_2) -> GND
- ESP32 pad 6: GND -> Net-(ACS2-Pin_2)
- ESP32 pad 7: Net-(ESP32-IO33) -> GND
- ESP32 pad 8: unconnected-(ESP32-IO25-Pad8) -> Net-(ESP32-IO25)
- R5 pad 2: Net-(ESP32-IO33) -> Net-(ESP32-IO25)
- R6 pad 1: Net-(ESP32-IO33) -> Net-(ESP32-IO25)
Routing:
- net GND: track 193.8 -> 0.04 mm
- net Net-(ESP32-IO33): track 47.8 -> 0.00 mm
- net Net-(ESP32-IO25): track 0.00 -> 45.6 mm
- net Net-(ACS1-Pin_1): track 187.4 -> 210.0 mm
- net Net-(MPPT1-Pad1): track 28.0 -> 38.0 mm
- net Net-(ESP32-IO12): track 73.0 -> 80.8 mm
- net Net-(PCB_Vin1-Pad1): track 27.0 -> 34.2 mm
- net Net-(ESP32-IO13): track 56.1 -> 60.5 mm
- net Net-(ADS1115-VDD): track 104.6 -> 108.6 mm
- net Net-(ACS2-Pin_2): track 18.9 -> 22.2 mm
- net Net-(ADS1115-A2): track 32.9 -> 30.4 mm
- net Net-(ACS3-Pin_2): track 9.38 -> 11.3 mm
- net Net-(PCB_Vin2-Pad1): track 29.4 -> 27.7 mm
- net Net-(ADS1115-SCL): track 31.6 -> 33.0 mm
- net Net-(ADS1115-A0): track 48.4 -> 47.9 mm
