File: _autosave-Telemetria_Hardware.kicad_pcb (KiCad board)
At the start: 2 copper layers, 27 parts, among them M100A1 1715734, SW1 RESET BUTTON, U1 CA3140, U2 CA3140

Commit message: teste4
Routing:
- net Net-(ADS1115-VDD): track 108.6 -> 110.6 mm
Changed lines of the file:
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@@
-	)
-	(segment
-		(start 104.917817 106.512183)
-		(end 107.95 103.48)
-		(width 0.8)
-		(layer "F.Cu")
-		(net 10)
 	)
 	(segment
@@
 	)
 	(segment
+		(start 75.946 66.04)
+		(end 76.2 66.04)
+		(width 0.8)
+		(layer "F.Cu")
+		(net 10)
+	)
+	(segment
+		(start 105.71 107.29)
+		(end 104.14 107.29)
+		(width 0.8)
+		(layer "F.Cu")
+		(net 10)
+	)
+	(segment
 		(start 102.21 109.22)
 		(end 104.14 107.29)
@@
 	)
 	(segment
-		(start 78.74 63.5)
-		(end 76.2 66.04)
-		(width 0.8)
-		(layer "F.Cu")
-		(net 10)
-	)
-	(segment
-		(start 107.95 103.48)
-		(end 107.95 69.85)
-		(width 0.8)
-		(layer "F.Cu")
-		(net 10)
-	)
-	(segment
-		(start 107.95 69.85)
-		(end 101.6 63.5)
+		(start 107.95 105.05)
+		(end 105.71 107.29)
 		(width 0.8)
 		(layer "F.Cu")
@@
 	)
 	(segment
-		(start 101.6 63.5)
+		(start 76.2 66.04)
 		(end 78.74 63.5)
+		(width 0.8)
+		(layer "F.Cu")
+		(net 10)
+	)
+	(segment
+		(start 78.74 63.5)
+		(end 101.6 63.5)
 		(width 0.8)
 		(layer "F.Cu")
@@
 	)
 	(segment
-		(start 76.2 66.04)
-		(end 75.946 66.04)
+		(start 101.6 63.5)
+		(end 107.95 69.85)
+		(width 0.8)
+		(layer "F.Cu")
+		(net 10)
+	)
+	(segment
+		(start 107.95 69.85)
+		(end 107.95 105.05)
 		(width 0.8)
 		(layer "F.Cu")
@@
 	)
 	(segment
-		(start 106 121)
-		(end 110.75 121)
+		(start 129.54 102.21)
+		(end 127.04 102.21)
 		(width 0.8)
 		(layer "F.Cu")
@@
 	)
 	(segment
-		(start 110.75 121)
-		(end 129.54 102.21)
-		(width 0.8)
-		(layer "F.Cu")
+		(start 127.04 102.21)
+		(end 108.25 121)
+		(width 0.8)
+		(layer "F.Cu")
+		(net 20)
+	)
+	(segment
+		(start 108.25 121)
+		(end 106 121)
+		(width 0.8)
+		(layer "F.Cu")
