File: Telemetria_Hardware.kicad_sch (KiCad schematic)
At the start: 16 parts, among them M100A1 1715734

Commit message: ads adicionado
Parts:
- ESP32: footprint esp32_devkit_v1_doit:esp32_devkit_v1_doit -> ESP32-DOIT-DEVKIT:ESP32-DOIT-DEVKIT

Commit message: placa teste
Parts:
- added ACS3: Conn_01x03_Female, Connector_PinSocket_2.54mm:PinSocket_1x03_P2.54mm_Vertical, symbol Connector:Conn_01x03_Female
- added PCB_Vin2, PCB_Vin3: CTB1202_2BK, TerminalBlock:TerminalBlock_bornier-2_P5.08mm, symbol KRE_Terminal_2Way_5.08mm:CTB1202_2BK
- added R10, R11, R5, R6, R7, R8, R9: R, Resistor_THT:R_Axial_DIN0207_L6.3mm_D2.5mm_P10.16mm_Horizontal, symbol Device:R
- added SW1: RESET BUTTON, symbol Switch:SW_MEC_5G
- B150A1, M100A1: footprint Terminal_Block_PCB_3Way:Connector_KRE_3W_5,08mm -> TerminalBlock:TerminalBlock_bornier-3_P5.08mm
- MPPT1, PCB_Vin1, STEP1: footprint Terminal_Block_PCB_2Way:KRE_Terminal_2Way_5.08mm -> TerminalBlock:TerminalBlock_bornier-2_P5.08mm
Connections:
- net GND: now also ACS3.3 (Pin_3), PCB_Vin2.2, PCB_Vin3.2, R10.2, R6.2, R8.2, SW1.3 (B), SW1.4 (B)
- net at ESP32.12 (IO12): now also R10.1, R11.1
- net at ESP32.13 (IO13): now also R8.1, R9.1
- net at ACS1.1 (Pin_1), ACS2.1 (Pin_1), B150A1.3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: now also ACS3.1 (Pin_1)
- net at ADS1115.1 (VDD), C2.1, DHT1.1 (Pin_1)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: now also R7.1
- net at ESP32.7 (IO33): now also R5.2, R6.1
- new net: PCB_Vin2.1, R9.2
- new net: PCB_Vin3.1, R11.2
- new net: R7.2, SW1.1 (A), SW1.2 (A)
- new net: ACS3.2 (Pin_2), R5.1
- no-connect marks 1 -> 18
Other:
- moved on the sheet: C1, STEP1

Commit message: teste 2
Parts:
- removed C2: C_Polarized, Capacitor_THT:C_Radial_D6.3mm_H11.0mm_P2.50mm, symbol Device:C_Polarized
- removed DHT1: Conn_01x04_Female, Connector_PinSocket_2.54mm:PinSocket_1x04_P2.54mm_Vertical, symbol Connector:Conn_01x04_Female
- removed R7: R, Resistor_THT:R_Axial_DIN0207_L6.3mm_D2.5mm_P10.16mm_Horizontal, symbol Device:R
- added R12: R, Resistor_THT:R_Axial_DIN0207_L6.3mm_D2.5mm_P10.16mm_Horizontal, symbol Device:R
- ESP32: footprint ESP32-DOIT-DEVKIT:ESP32-DOIT-DEVKIT -> ESP32:esp32_devkit_v1_doit
- SW1: footprint (none) -> BUTT:BUTT
Connections:
- net GND: now also ESP32.6 (IO32), R12.2; no longer SW1.3 (B), SW1.4 (B)
- net at ADS1115.1 (VDD), ESP32.16 (3V3): now also ESP32.20 (IO4), SW1.1 (A), SW1.2 (A), SW1.3 (B), SW1.4 (B), R12.1
- no-connect marks 18 -> 16
Other:
- moved on the sheet: ACS1, ACS2, ACS3, ADS1115, B150A1, C1, ESP32, M100A1, MPPT1, PCB_Vin1, PCB_Vin2, PCB_Vin3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

Commit message: teste4
Parts:
- added U1, U2: CA3140, Package_DIP:DIP-8_W7.62mm_Socket_LongPads, symbol Amplifier_Operational:CA3140
Connections:
- net GND: now also ESP32.5 (IO35), ESP32.7 (IO33), U1.4 (V-), U2.4 (V-); no longer ESP32.6 (IO32), PCB_Vin2.2, PCB_Vin3.2
- net at ESP32.12 (IO12), R11.1: no longer R10.1
- net at ESP32.13 (IO13), R9.1: no longer R8.1
- net at ACS2.2 (Pin_2): now also ESP32.6 (IO32); no longer ESP32.5 (IO35)
- net at R5.2, R6.1: now also ESP32.8 (IO25); no longer ESP32.7 (IO33)
- net at PCB_Vin2.1: now also U1.2 (-); no longer R9.2
- net at R11.2: now also R10.1, U2.6; no longer PCB_Vin3.1
- new net: PCB_Vin2.2, U1.3 (+), U1.7 (V+)
- new net: R8.1, R9.2, U1.6
- new net: PCB_Vin3.1, U2.2 (-)
- new net: PCB_Vin3.2, U2.3 (+), U2.7 (V+)
- no-connect marks 16 -> 15
Other:
- note added: "3,3V??"
- note added: "Package_DIP:DIP-8_W7.62mm_Socket_LongPads footprint ampop"
- note added: "procurar saber se tem que passar apenas 3,3V para o esp e fazer os calculos dos restistores responsaveis pelo divisor de tensão"
- moved on the sheet: PCB_Vin2, PCB_Vin3, R10, R11, R8, R9

Commit message: upp
Parts:
- removed SW1: RESET BUTTON, BUTT:BUTT, symbol Switch:SW_MEC_5G
- added SW1: SW_SPST, Button_Switch_THT:SW_DIP_SPSTx01_Slide_9.78x4.72mm_W7.62mm_P2.54mm, symbol Switch:SW_SPST
Connections:
- net at ADS1115.1 (VDD), ESP32.16 (3V3): now also SW1.1 (A); no longer ESP32.20 (IO4), R12.1
- new net: ESP32.20 (IO4), R12.1, SW1.2 (B)
Changed lines of the file:
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@@
 	)
 	(junction
-		(at 60.96 22.86)
-		(diameter 0)
-		(color 0 0 0 0)
-	)
-	(junction
 		(at 127 110.49)
 		(diameter 0)
@@
 	)
 	(junction
-		(at 50.8 22.86)
-		(diameter 0)
-		(color 0 0 0 0)
-	)
-	(junction
 		(at 127 137.16)
 		(diameter 0)
@@
 	(wire
 		(pts
-			(xy 50.8 22.86) (xy 60.96 22.86)
-		)
-		(stroke
-			(width 0)
-			(type default)
-		)
-	)
-	(wire
-		(pts
 			(xy 227.33 82.55) (xy 233.68 82.55)
 		)
@@
 	)
 	(symbol
-		(lib_id "Switch:SW_MEC_5G")
-		(at 55.88 22.86 0)
-		(unit 1)
-		(exclude_from_sim no)
-		(in_bom yes)
-		(on_board yes)
-		(dnp no)
-		(property "Reference" "SW1"
-			(at 55.88 16.51 0)
-			(effects
-				(font
-					(size 1.27 1.27)
-				)
-			)
-		)
-		(property "Value" "RESET BUTTON"
-			(at 55.88 19.05 0)
-			(effects
-				(font
-					(size 1.27 1.27)
-				)
-			)
-		)
-		(property "Footprint" "BUTT:BUTT"
-			(at 55.88 17.78 0)
-			(effects
-				(font
-					(size 1.27 1.27)
-				)
-				(hide yes)
-			)
-		)
-		(property "Datasheet" "http://www.apem.com/int/index.php?controller=attachment&id_attachment=488"
-			(at 55.88 17.78 0)
-			(effects
-				(font
-					(size 1.27 1.27)
-				)
-				(hide yes)
-			)
-		)
-		(property "Description" ""
-			(at 55.88 22.86 0)
-			(effects
-				(font
-					(size 1.27 1.27)
-				)
-				(hide yes)
-			)
-		)
-		(pin "1"
-		)
-		(pin "2"
-		)
-		(pin "4"
-		)
-		(pin "3"
-		)
-		(instances
-			(project "Telemetria_Hardware"
-				(path "/c806ca64-4076-499b-9029-155759542c55"
-					(reference "SW1")
-					(unit 1)
-				)
-			)
-		)
-	)
-	(symbol
 		(lib_id "Amplifier_Operational:CA3140")
 		(at 251.46 43.18 180)
@@
 					(unit 1)
 				)
+			)
+		)
+	)
+	(symbol
+		(lib_id "Switch:SW_SPST")
+		(at 55.88 22.86 0)
+		(unit 1)
+		(exclude_from_sim no)
+		(in_bom yes)
+		(on_board yes)
+		(dnp no)
+		(fields_autoplaced yes)
+		(property "Reference" "SW1"
+			(at 55.88 16.51 0)
+			(effects
+				(font
+					(size 1.27 1.27)
+				)
+			)
+		)
+		(property "Value" "SW_SPST"
+			(at 55.88 19.05 0)
+			(effects
+				(font
+					(size 1.27 1.27)
+				)
+			)
+		)
+		(property "Footprint" "Button_Switch_THT:SW_DIP_SPSTx01_Slide_9.78x4.72mm_W7.62mm_P2.54mm"
+			(at 55.88 22.86 0)
+			(effects
+				(font
+					(size 1.27 1.27)
+				)
+				(hide yes)
+			)
+		)
+		(property "Datasheet" "~"
+			(at 55.88 22.86 0)
+			(effects
+				(font
+					(size 1.27 1.27)
+				)
+				(hide yes)
+			)
+		)
+		(property "Description" "Single Pole Single Throw (SPST) switch"
+			(at 55.88 22.86 0)
+			(effects
+				(font
+					(size 1.27 1.27)
+				)
+				(hide yes)
+			)
+		)
+		(pin "2"
+		)
+		(pin "1"
+		)
+		(instances
+			(project "Telemetria_Hardware"
+				(path "/c806ca64-4076-499b-9029-155759542c55"
+					(reference "SW1")
+					(unit 1)
+				)
