File: Telemetria_Hardware.kicad_sch (KiCad schematic)
At the start: 16 parts, among them M100A1 1715734

Commit message: Mudanças pré DSB 2024
Parts:
- removed C2: C_Polarized, Capacitor_THT:C_Radial_D6.3mm_H11.0mm_P2.50mm, symbol Device:C_Polarized
- removed DHT1: Conn_01x04_Female, Connector_PinSocket_2.54mm:PinSocket_1x04_P2.54mm_Vertical, symbol Connector:Conn_01x04_Female
- removed ESP32: ESP32_DevKit_V1_DOIT, esp32_devkit_v1_doit:esp32_devkit_v1_doit, symbol esp32_devkit_v1_doit:ESP32_DevKit_V1_DOIT
- added ESP1: ESP32_DevKit_V1_DOIT, ESP32:esp32_devkit_v1_doit, symbol esp32_devkit_v1_doit:ESP32_DevKit_V1_DOIT
- added PCB_Vin3, STEP2: CTB1202_2BK, TerminalBlock:TerminalBlock_bornier-2_P5.08mm, symbol KRE_Terminal_2Way_5.08mm:CTB1202_2BK
- added Q2: TIP120, Package_TO_SOT_THT:TO-220-3_Vertical, symbol Transistor_BJT:TIP120
- added R10: 130Ω, Resistor_THT:R_Axial_DIN0207_L6.3mm_D2.5mm_P10.16mm_Horizontal, symbol Device:R
- added R12: R, Resistor_THT:R_Axial_DIN0207_L6.3mm_D2.5mm_P10.16mm_Horizontal, symbol Device:R
- added R9: 39Ω, Resistor_THT:R_Axial_DIN0207_L6.3mm_D2.5mm_P10.16mm_Horizontal, symbol Device:R
- added SW1: SW_SPST, Button_Switch_THT:SW_DIP_SPSTx01_Slide_9.78x4.72mm_W7.62mm_P2.54mm, symbol Switch:SW_SPST
- B150A1, M100A1: footprint Terminal_Block_PCB_3Way:Connector_KRE_3W_5,08mm -> TerminalBlock:TerminalBlock_bornier-3_P5.08mm
- MPPT1, PCB_Vin1, STEP1: footprint Terminal_Block_PCB_2Way:KRE_Terminal_2Way_5.08mm -> TerminalBlock:TerminalBlock_bornier-2_P5.08mm
Connections:
- net GND: now also R2.2, ESP1.14 (GND), ESP1.17 (GND), R10.2, R12.2; no longer R2.1
- net at ACS1.1 (Pin_1), ACS2.1 (Pin_1), B150A1.3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: now also ESP1.15 (VIN)
- net at ADS1115.1 (VDD): now also ESP1.16 (3V3), SW1.1 (A)
- net at R1.1: now also R2.1, ESP1.21 (IO16); no longer R2.2
- net at ADS1115.4 (SDA): now also ESP1.26 (IO21)
- net at ADS1115.3 (SCL): now also ESP1.29 (IO22)
- net at ACS1.2 (Pin_2): now also ESP1.4 (IO34)
- net at ACS2.2 (Pin_2): now also ESP1.6 (IO32)
- net at ADS1115.10 (A3): now also R10.1, R9.1
- new net: Q2.2 (C), R9.2
- new net: ESP1.20 (IO4), R12.1, SW1.2 (B)
- new net: PCB_Vin3.2, Q2.1 (B)
- new net: PCB_Vin3.1, Q2.3 (E)
- new net: ESP1.5 (IO35), STEP2.1
- new net: ESP1.7 (IO33), STEP2.2
- no-connect marks 1 -> 11
Other:
- note added: "0-3.3076V"
- note added: "Polo possitivo do Pot"
- note added: "procurar saber se tem que passar apenas 3,3V para o esp e fazer os calculos dos restistores responsaveis pelo divisor de tensão"
- moved on the sheet: ADS1115, B150A1, M100A1, MPPT1, PCB_Vin1, STEP1

Commit message: Mudanças Pré DSB/2
Other:
- note added: "Ios 33 é o fio do bateria"
Changed lines of the file:
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@@
+		)
+	)
+	(text "Ios 33 é o fio do bateria"
+		(exclude_from_sim no)
+		(at 77.724 158.75 0)
+		(effects
+			(font
+				(size 1.27 1.27)
+			)
 		)
 	)
@@
 		)
 	)
-	(label "Ios 33 é o fio do bateria"
-		(at 66.04 158.75 0)
-		(fields_autoplaced yes)
-		(effects
-			(font
-				(size 1.27 1.27)
-			)
-			(justify left bottom)
-		)
-	)
